Commit message: match params with the good policy

File: resources/robots/mevius/urdf/mevius.urdf (robot description, URDF)
Before this commit: robot mevius, 13 links, 12 joints
Links:
- added link BL_foot_link, mass 0.05; collision sphere radius=0.025; visual sphere radius=0.025
- added link BR_foot_link, mass 0.05; collision sphere radius=0.025; visual sphere radius=0.025
- added link FL_foot_link, mass 0.05; collision sphere radius=0.025; visual sphere radius=0.025
- added link FR_foot_link, mass 0.05; collision sphere radius=0.025; visual sphere radius=0.025
- link BL_calf_link: mass 0.0819657771505335 -> 0.101512760080133; geometry collision cylinder length=0.23 radius=0.01; visual mesh filename=../meshes/BL_calf_link.STL
- link BL_scapula_link: geometry collision cylinder length=0.08 radius=0.05; visual mesh filename=../meshes/BL_scapula_link.STL
- link BL_thigh_link: geometry visual mesh filename=../meshes/BL_thigh_link.STL
- link BR_calf_link: mass 0.081966 -> 0.101512760080133; geometry collision cylinder length=0.23 radius=0.01; visual mesh filename=../meshes/BR_calf_link.STL
- link BR_scapula_link: geometry collision cylinder length=0.08 radius=0.05; visual mesh filename=../meshes/BR_scapula_link.STL
- link BR_thigh_link: mass 1.2804 -> 1.28036049228712; geometry visual mesh filename=../meshes/BR_thigh_link.STL
- link FL_calf_link: mass 0.081966 -> 0.101512760080133; geometry collision cylinder length=0.23 radius=0.01; visual mesh filename=../meshes/FL_calf_link.STL
- link FL_scapula_link: mass 0.792389082205849 -> 0.79238908220585; geometry collision cylinder length=0.08 radius=0.05; visual mesh filename=../meshes/FL_scapula_link.STL
- link FL_thigh_link: geometry visual mesh filename=../meshes/FL_thigh_link.STL
- link FR_calf_link: mass 0.081966 -> 0.101512760080133; geometry collision cylinder length=0.23 radius=0.01; visual mesh filename=../meshes/FR_calf_link.STL
- link FR_scapula_link: geometry collision cylinder length=0.08 radius=0.05; visual mesh filename=../meshes/FR_scapula_link.STL
- link FR_thigh_link: geometry visual mesh filename=../meshes/FR_thigh_link.STL
- link base_link: mass 7.46950563423809 -> 8.0; geometry collision box size=0.334 0.200 0.150; visual mesh filename=../meshes/base_link.STL
Joints:
- added joint BL_ankle_joint: type fixed, parent BL_calf_link, child BL_foot_link, origin xyz=0.003 0.0 -0.235 rpy=0 0 0
- added joint BR_ankle_joint: type fixed, parent BR_calf_link, child BR_foot_link, origin xyz=0.003 0.0 -0.235 rpy=0 0 0
- added joint FL_ankle_joint: type fixed, parent FL_calf_link, child FL_foot_link, origin xyz=0.003 0.0 -0.235 rpy=0 0 0
- added joint FR_ankle_joint: type fixed, parent FR_calf_link, child FR_foot_link, origin xyz=0.003 0.0 -0.235 rpy=0 0 0
- joint BL_collar: limit lower=-0.7854 upper=0.7854 effort=25 velocity=500 -> lower=-0.7854 upper=0.7854 effort=25 velocity=310
- joint BL_hip: limit lower=-1.5708 upper=1.5708 effort=25 velocity=500 -> lower=0.0 upper=2.0944 effort=25 velocity=310
- joint BL_knee: limit lower=-2.8856 upper=-1.0 effort=25 velocity=500 -> lower=-2.8745 upper=-1.08 effort=25 velocity=310
- joint BR_collar: limit lower=-0.7854 upper=0.7854 effort=25 velocity=500 -> lower=-0.7854 upper=0.7854 effort=25 velocity=310
- joint BR_hip: limit lower=-1.5708 upper=1.5708 effort=25 velocity=500 -> lower=0.0 upper=2.0944 effort=25 velocity=310
- joint BR_knee: limit lower=-2.8856 upper=-1.0 effort=25 velocity=500 -> lower=-2.8745 upper=-1.08 effort=25 velocity=310; origin xyz=0 -0.0655500000000101 -0.249999999999997 rpy=0 0 0 -> xyz=0 -0.06555 -0.25 rpy=0 0 0
- joint FL_collar: limit lower=-0.7854 upper=0.7854 effort=25 velocity=500 -> lower=-0.7854 upper=0.7854 effort=25 velocity=310; origin xyz=0.16405000000001 0.0719999999999999 0.0565000346699527 rpy=0 0 0 -> xyz=0.16405000000001 0.0720000000000002 0.056500000000002 rpy=0 0 0
- joint FL_hip: limit lower=-1.5708 upper=1.5708 effort=25 velocity=500 -> lower=0.0 upper=2.0944 effort=25 velocity=310; origin xyz=0.0555000000000055 0.01205000000001 0 rpy=0 0 0 -> xyz=0.0555000000000021 0.01205000000001 0 rpy=0 0 0
- joint FL_knee: limit lower=-2.8856 upper=-1.0 effort=25 velocity=500 -> lower=-2.8745 upper=-1.08 effort=25 velocity=310; origin xyz=0 0.06555000000001 -0.249999999999998 rpy=0 0 0 -> xyz=0 0.06555000000001 -0.250000000000004 rpy=0 0 0
- joint FR_collar: limit lower=-0.7854 upper=0.7854 effort=25 velocity=500 -> lower=-0.7854 upper=0.7854 effort=25 velocity=310
- joint FR_hip: limit lower=-1.5708 upper=1.5708 effort=25 velocity=500 -> lower=0.0 upper=2.0944 effort=25 velocity=310
- joint FR_knee: limit lower=-2.8856 upper=-1.0 effort=25 velocity=500 -> lower=-2.8745 upper=-1.08 effort=25 velocity=310
