Commit message: モータ付きモデルに対応した

File: resources/robots/ramiel2/urdf/ramiel2_tendon.urdf (robot description, URDF)
Before this commit: robot ramiel2, 22 links, 21 joints
Joints:
- joint motor_0: limit (none) -> effort=10 velocity=2000
- joint motor_1: limit (none) -> effort=10 velocity=2000
- joint motor_2: limit (none) -> effort=10 velocity=2000
- joint motor_3: limit (none) -> effort=10 velocity=2000
- joint motor_4: limit (none) -> effort=10 velocity=2000
- joint motor_5: limit (none) -> effort=10 velocity=2000

Commit message: モーターが回るようになった

File: resources/robots/ramiel2/urdf/ramiel2_tendon.urdf (robot description, URDF)
Before this commit: robot ramiel2, 22 links, 21 joints
Links:
- link motor_0_link: geometry visual mesh filename=../meshes/motor_0_link.STL
- link motor_1_link: geometry visual mesh filename=../meshes/motor_1_link.STL
- link motor_2_link: geometry visual mesh filename=../meshes/motor_2_link.STL
- link motor_3_link: geometry visual mesh filename=../meshes/motor_3_link.STL
- link motor_4_link: geometry visual mesh filename=../meshes/motor_4_link.STL
- link motor_5_link: geometry visual mesh filename=../meshes/motor_5_link.STL
Joints:
- joint motor_0: type continuous -> revolute
- joint motor_1: type continuous -> revolute
- joint motor_2: type continuous -> revolute
- joint motor_3: type continuous -> revolute
- joint motor_4: type continuous -> revolute
- joint motor_5: type continuous -> revolute
