Commit message: armatureと直動関節のlimitを正しくした

File: resources/robots/ramiel2/urdf/ramiel2.urdf (robot description, URDF)
Before this commit: robot ramiel2, 4 links, 3 joints
Joints:
- joint slide: limit lower=-0.5 upper=0.5 effort=1500 velocity=20 -> lower=-0.4195 upper=0.4195 effort=1500 velocity=20

Commit message: stiffnes, damping, reward調整. torque_limit変更

File: resources/robots/ramiel2/urdf/ramiel2.urdf (robot description, URDF)
Before this commit: robot ramiel2, 4 links, 3 joints
Joints:
- joint pitch: limit lower=-0.69813170079 upper=0.69813170079 effort=150 velocity=500 -> lower=-0.69813170079 upper=0.69813170079 effort=100 velocity=500
- joint roll: limit lower=-0.69813170079 upper=0.69813170079 effort=150 velocity=500 -> lower=-0.69813170079 upper=0.69813170079 effort=100 velocity=500
- joint slide: limit lower=-0.4195 upper=0.4195 effort=1500 velocity=20 -> lower=-0.4195 upper=0.4195 effort=1000 velocity=20

Commit message: tendon_model_gym追加. TendonRobotModel初期化できた

File: resources/robots/ramiel2/urdf/ramiel2.urdf (robot description, URDF)
Before this commit: robot ramiel2, 4 links, 3 joints
Links:
- added link env_link, mass 0.0001
- added link point_base_0_0, mass 3.41805280710569E-05; visual mesh filename=../meshes/point_base_0_0.STL
- added link point_base_1_0, mass 3.41805280710569E-05; visual mesh filename=../meshes/point_base_1_0.STL
- added link point_base_2_0, mass 3.41805280710569E-05; visual mesh filename=../meshes/point_base_2_0.STL
- added link point_base_3_0, mass 3.41805280710569E-05; visual mesh filename=../meshes/point_base_3_0.STL
- added link point_base_4_0, mass 3.41805280710569E-05; visual mesh filename=../meshes/point_base_4_0.STL
- added link point_base_5_0, mass 3.41805280710569E-05; visual mesh filename=../meshes/point_base_5_0.STL
- added link point_leg_0_1, mass 3.41805280710569E-05; visual mesh filename=../meshes/point_leg_0_1.STL
- added link point_leg_1_1, mass 3.4181E-05; visual mesh filename=../meshes/point_leg_1_1.STL
- added link point_leg_2_1, mass 3.41805280710569E-05; visual mesh filename=../meshes/point_leg_2_1.STL
- added link point_leg_3_1, mass 3.41805280710569E-05; visual mesh filename=../meshes/point_leg_3_1.STL
- added link point_leg_4_1, mass 3.41805280710569E-05; visual mesh filename=../meshes/point_leg_4_1.STL
- added link point_leg_5_1, mass 3.41805280710569E-05; visual mesh filename=../meshes/point_leg_5_1.STL
Joints:
- added joint joint_floating: type floating, parent env_link, child base_link, origin xyz=0 0 0 rpy=0 0 0
- added joint point_base_0_0_dummy: type fixed, parent base_link, child point_base_0_0, origin xyz=0.32 0 0.03 rpy=0 0 0, axis 0 0 0
- added joint point_base_1_0_dummy: type fixed, parent base_link, child point_base_1_0, origin xyz=-0.16 0.27713 0.03 rpy=0 0 0, axis 0 0 0
- added joint point_base_2_0_dummy: type fixed, parent base_link, child point_base_2_0, origin xyz=-0.16 -0.27713 0.03 rpy=0 0 0, axis 0 0 0
- added joint point_base_3_0_dummy: type fixed, parent base_link, child point_base_3_0, origin xyz=0.32 0 -0.0299999999999999 rpy=0 0 0, axis 0 0 0
- added joint point_base_4_0_dummy: type fixed, parent base_link, child point_base_4_0, origin xyz=-0.16 0.27713 -0.03 rpy=0 0 0, axis 0 0 0
- added joint point_base_5_0_dummy: type fixed, parent base_link, child point_base_5_0, origin xyz=-0.16 -0.27713 -0.03 rpy=0 0 0, axis 0 0 0
- added joint point_leg_0_1_dummy: type fixed, parent leg_link, child point_leg_0_1, origin xyz=0.024 0 0.52 rpy=0 0 0, axis 0 0 0
- added joint point_leg_1_1_dummy: type fixed, parent leg_link, child point_leg_1_1, origin xyz=-0.012 0.020785 0.52 rpy=0 0 0, axis 0 0 0
- added joint point_leg_2_1_dummy: type fixed, parent leg_link, child point_leg_2_1, origin xyz=-0.012 -0.0207846096908265 0.52 rpy=0 0 0, axis 0 0 0
- added joint point_leg_3_1_dummy: type fixed, parent leg_link, child point_leg_3_1, origin xyz=0.024 0 -0.52 rpy=0 0 0, axis 0 0 0
- added joint point_leg_4_1_dummy: type fixed, parent leg_link, child point_leg_4_1, origin xyz=-0.0120000000000001 0.0207846096908265 -0.52 rpy=0 0 0, axis 0 0 0
- added joint point_leg_5_1_dummy: type fixed, parent leg_link, child point_leg_5_1, origin xyz=-0.012 -0.020785 -0.52 rpy=0 0 0, axis 0 0 0

Commit message: urdfにモーター追加. まだmotorとjointでプログラムを分岐できてないからエラーでる

File: resources/robots/ramiel2/urdf/ramiel2.urdf (robot description, URDF)
Before this commit: robot ramiel2, 17 links, 16 joints
Links:
- removed link env_link
- added link motor_0_link, mass 0.0001; collision mesh filename=../meshes/motor_0_link.STL; visual mesh filename=../meshes/motor_0_link.STL
- added link motor_1_link, mass 0.0001; collision mesh filename=../meshes/motor_1_link.STL; visual mesh filename=../meshes/motor_1_link.STL
- added link motor_2_link, mass 0.0001; collision mesh filename=../meshes/motor_2_link.STL; visual mesh filename=../meshes/motor_2_link.STL
- added link motor_3_link, mass 0.0001; collision mesh filename=../meshes/motor_3_link.STL; visual mesh filename=../meshes/motor_3_link.STL
- added link motor_4_link, mass 0.0001; collision mesh filename=../meshes/motor_4_link.STL; visual mesh filename=../meshes/motor_4_link.STL
- added link motor_5_link, mass 0.0001; collision mesh filename=../meshes/motor_5_link.STL; visual mesh filename=../meshes/motor_5_link.STL
Joints:
- removed joint joint_floating
- added joint motor_0: type continuous, parent base_link, child motor_0_link, origin xyz=-0.019259 -0.23197 0.00725 rpy=0 0 2.1468, axis -1 0 0
- added joint motor_1: type continuous, parent base_link, child motor_1_link, origin xyz=0.21052 0.099308 0.00725 rpy=0 0 -2.042, axis -1 0 0
- added joint motor_2: type continuous, parent base_link, child motor_2_link, origin xyz=-0.19127 0.13266 0.00725 rpy=0 0 0, axis -0.99863 -0.052336 0
- added joint motor_3: type continuous, parent base_link, child motor_3_link, origin xyz=-0.019259 0.23197 -0.00725 rpy=0 0 -2.1468, axis -1 0 0
- added joint motor_4: type continuous, parent base_link, child motor_4_link, origin xyz=-0.19127 -0.13266 -0.00725 rpy=0 0 0, axis -0.99863 0.052336 0
- added joint motor_5: type continuous, parent base_link, child motor_5_link, origin xyz=0.210523758501758 -0.0993079211435383 -0.00724999999999996 rpy=0 0 2.04203522483338, axis -1 0 0

Commit message: urdfのcollisionを実機に近づけた. only positive rewardsをfalseにしてrewardを調節した. torque_convert_netをmintension120Nのものに変更した

File: resources/robots/ramiel2/urdf/ramiel2.urdf (robot description, URDF)
Before this commit: robot ramiel2, 17 links, 16 joints
Links:
- link base_link: geometry collision cylinder length=0.29 radius=0.04; collision cylinder length=0.29 radius=0.04
- link leg_link: geometry collision cylinder length=1.064 radius=0.033; visual mesh filename=../meshes/leg_link.STL

File: resources/robots/ramiel2/urdf/ramiel2_tendon.urdf (robot description, URDF)
Before this commit: robot ramiel2, 22 links, 21 joints
Links:
- link base_link: geometry collision cylinder length=0.29 radius=0.04; collision cylinder length=0.29 radius=0.04
- link leg_link: geometry collision cylinder length=1.064 radius=0.033; visual mesh filename=../meshes/leg_link.STL
